File: VT.kicad_pcb (KiCad board)
At the start: 2 copper layers, 433.3 x 119 mm, 434 parts, among them K1 KEYSW, K10 KEYSW, K100 KEYSW, K101 KEYSW, K102 KEYSW, K103 KEYSW, K104 KEYSW, K11 KEYSW, K12 KEYSW, K13 KEYSW, K14 KEYSW, K15 KEYSW, K16 KEYSW, K17 KEYSW, K18 KEYSW, K2 KEYSW, K20 KEYSW, K21 KEYSW, K22 KEYSW, K23 KEYSW, K24 KEYSW, K25 KEYSW, K26 KEYSW, K27 KEYSW, K28 KEYSW, K29 KEYSW, K3 KEYSW, K30 KEYSW, K31 KEYSW, K32 KEYSW, K33 KEYSW, K34 KEYSW, K35 KEYSW, K36 KEYSW, K37 KEYSW, K38 KEYSW, K39 KEYSW, K4 KEYSW, K40 KEYSW, K41 KEYSW, K42 KEYSW, K43 KEYSW, K44 KEYSW, K45 KEYSW, K46 KEYSW, K47 KEYSW, K48 KEYSW, K49 KEYSW, K5 KEYSW, K50 KEYSW, K51 KEYSW, K52 KEYSW, K53 KEYSW, K54 KEYSW, K55 KEYSW, K56 KEYSW, K57 KEYSW, K58 KEYSW, K59 KEYSW, K6 KEYSW, K60 KEYSW, K61 KEYSW, K62 KEYSW, K63 KEYSW, K64 KEYSW, K65 KEYSW, K66 KEYSW, K67 KEYSW, K68 KEYSW, K69 KEYSW, K7 KEYSW, K70 KEYSW, K71 KEYSW, K72 KEYSW, K73 KEYSW, K74 KEYSW, K75 KEYSW, K76 KEYSW, K77 KEYSW, K78 KEYSW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

Commit message: Fixed Issues
Parts:
- SW1: footprint Button_Switch_SMD:SW_SPDT_CK-JS102011SAQN -> Button_Switch_THT:SW_CuK_JS202011AQN_DPDT_Angled
- moved SW1 2.80 mm to (546.9, 98.6)
- renumbered Ke to K19
Routing:
- net GND: track 113.5 -> 108.8 mm, vias 1 -> 0
- net Net-(D105-Pad1): track 2507.4 -> 2509.2 mm
Other:
- board text added: "By Neil Feagan"
- board text removed: "By Hybrid65"

Commit message: Update VT.kicad_pcb
Other:
- board text added: "+"
Changed lines of the file:
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@@
-(kicad_pcb (version 20171130) (host pcbnew "(5.1.2)-1")
+(kicad_pcb (version 20171130) (host pcbnew "(5.1.5)-3")
   (general
     (thickness 1.6)
@@
     (effects (font (size 1.5 1.5) (thickness 0.3)))
   )
-  (gr_text enter (at 187.15 99.1369) (layer F.SilkS)
+  (gr_text + (at 187.15 99.1369) (layer F.SilkS)
     (effects (font (size 1.5 1.5) (thickness 0.3)))
   )
